File: sch/nlpgen/nlpgen.kicad_sch (KiCad schematic)
At the start: 16 parts, among them J1 vcc, J2 gnd, J3 nlp_disa, J4 sck, J5 mosi, J6 out, U1 74HC14, U2 74HCT86

Commit message: NLP generator board
Parts:
- C1, C2, C3, C4: footprint (none) -> Capacitor_SMD:C_0805_2012Metric
- J1, J2, J3, J4, J5, J6: footprint (none) -> Connector_Wire:SolderWire-0.5sqmm_1x01_D0.9mm_OD2.3mm_Relief
- J7, J8: renamed from J?; footprint (none) -> Connector_Wire:SolderWire-0.5sqmm_1x01_D0.9mm_OD2.3mm_Relief
- R1: footprint (none) -> Resistor_THT:R_Axial_DIN0204_L3.6mm_D1.6mm_P7.62mm_Horizontal
- R2: footprint (none) -> Resistor_SMD:R_0805_2012Metric
- U1: footprint (none) -> Package_SO:SOIC-14_3.9x8.7mm_P1.27mm
- U2: footprint (none) -> Package_DIP:DIP-14_W7.62mm
Connections:
- net GND: now also U1.5
- net VCC: now also U1.13
- net at U1.10: now also U1.9
- net at U1.11: now also U1.12
- no-connect marks 0 -> 2
Other:
- moved on the sheet: U1D, U1E, U1F
