File: sch/transmitter/transmitter.kicad_pcb (KiCad board)
At the start: 2 copper layers, 51 x 45.5 mm, 22 parts, among them J1 VCC, J2 VCC, J3 GND, J4 GND, J5 sck_tx, J6 mosi_tx, J7 driver_in, J8 driver_ena, Q1 2N7002, U1 74HCT86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

Commit message: Fix NLP polarity
Parts:
- C4: value ? -> 200
- C5: value 330 -> 200
- R1: value ? -> 560
- R3: value 300 -> 560
Connections:
- U1 pad 5: VCC -> GND
Routing:
- net VCC: track 126.9 -> 122.0 mm
