File: sch/shield/shield.kicad_pcb (KiCad board)
At the start: 4 copper layers, 69 x 74 mm, 60 parts, among them J1 ARJM11D7-009-AB-EW2, J2 partial-nucleo64, Q1 2N7002, Q2 2N7002, Q3 2N7002, SW1 invert, U1 74HC86, U2 74HC14, U3 75C1168, U4 74HC08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

Commit message: Fix error in board
Parts:
- C10: value 10 -> 12
- C13: value 0.1 -> 0.68
- R10, R9: value 330 -> 150
- R5: value 500 -> 560
- R7: value 500k -> 57.6k
- TP3: value edge delay -> TestPoint
Connections:
- U8 pad 2: /sck_tx -> GND
Routing:
- net GND: track 45.2 -> 46.8 mm, vias 34 -> 35
- net /sck_tx: track 22.9 -> 21.5 mm
Other:
- board text added: "EthSh rev.2"
- board text removed: "EthSh rev.1"
Changed lines of the file:
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@@
   (title_block
     (title "Ethernet to SPI adapter, Nucleo-64 shield")
-    (date "2022-11-16")
-    (rev "1")
+    (date "2022-11-25")
+    (rev "2")
     (comment 1 "Licensed under the TAPR Open Hardware License (www.tapr.org/OHL)")
   )
@@
       (effects (font (size 1 1) (thickness 0.15)))
     )
-    (fp_text value "330" (at 0 1.65 90) (layer "F.Fab")
+    (fp_text value "150" (at 0 1.65 90) (layer "F.Fab")
       (effects (font (size 1 1) (thickness 0.15)))
     )
@@
       (net 25 "/sck_tx") (pintype "input"))
     (pad "2" smd roundrect (at -2.475 -2.54) (size 1.95 0.6) (layers "F.Cu" "F.Paste" "F.Mask") (roundrect_rratio 0.25)
-      (net 25 "/sck_tx") (pintype "input"))
+      (net 2 "GND") (pintype "input"))
     (pad "3" smd roundrect (at -2.475 -1.27) (size 1.95 0.6) (layers "F.Cu" "F.Paste" "F.Mask") (roundrect_rratio 0.25)
       (net 31 "Net-(Q3-Pad1)") (pintype "output"))
@@
       (effects (font (size 1 1) (thickness 0.15)))
     )
-    (fp_text value "edge delay" (at -3.1 1.75) (layer "F.SilkS")
+    (fp_text value "TestPoint" (at -3.1 1.75) (layer "F.SilkS")
       (effects (font (size 1 1) (thickness 0.15)))
     )
@@
       (effects (font (size 1 1) (thickness 0.15)))
     )
-    (fp_text value "0.1" (at 0 1.68) (layer "F.Fab")
+    (fp_text value "0.68" (at 0 1.68) (layer "F.Fab")
       (effects (font (size 1 1) (thickness 0.15)))
     )
@@
       (effects (font (size 1 1) (thickness 0.15)))
     )
-    (fp_text value "500k" (at 3.75 0.2) (layer "F.Fab")
+    (fp_text value "57.6k" (at 3.75 0.2) (layer "F.Fab")
       (effects (font (size 1 1) (thickness 0.15)))
     )
@@
       (effects (font (size 1 1) (thickness 0.15)))
     )
-    (fp_text value "10" (at -0.1 3.1) (layer "F.Fab")
+    (fp_text value "12" (at -0.1 3.1) (layer "F.Fab")
       (effects (font (size 1 1) (thickness 0.15)))
     )
@@
       (effects (font (size 1 1) (thickness 0.15)))
     )
-    (fp_text value "500" (at 0 1.65 90) (layer "F.Fab")
+    (fp_text value "560" (at 0 1.65 90) (layer "F.Fab")
       (effects (font (size 1 1) (thickness 0.15)))
     )
@@
       (effects (font (size 1 1) (thickness 0.15)))
     )
-    (fp_text value "330" (at 0 1.65 90) (layer "F.Fab")
+    (fp_text value "150" (at 0 1.65 90) (layer "F.Fab")
       (effects (font (size 1 1) (thickness 0.15)))
     )
@@
   (gr_arc (start 81 67.5) (mid 77.636594 66.20934) (end 76 63) (layer "Edge.Cuts") (width 0.1))
   (gr_line (start 61 137) (end 61 63) (layer "Edge.Cuts") (width 0.1))
-  (gr_text "EthSh rev.1" (at 79 135) (layer "F.Cu")
+  (gr_text "EthSh rev.2" (at 79 135) (layer "F.Cu")
     (effects (font (size 1 1) (thickness 0.2)))
   )
@@
   (segment (start 64 123) (end 64 121) (width 0.3) (layer "F.Cu") (net 2))
   (segment (start 99.35 89.6) (end 98.4 89.6) (width 0.15) (layer "F.Cu") (net 2))
+  (segment (start 72.725 74.16) (end 71.16 74.16) (width 0.3) (layer "F.Cu") (net 2))
   (segment (start 111.75 132.445) (end 111.75 133.25) (width 0.3) (layer "F.Cu") (net 2))
   (segment (start 63.725 83.3) (end 64.8 83.3) (width 0.3) (layer "F.Cu") (net 2))
@@
   (segment (start 85.7375 102.3625) (end 85.7 102.4) (width 0.3) (layer "F.Cu") (net 2))
   (segment (start 102.7625 95.05) (end 103.95 95.05) (width 0.3) (layer "F.Cu") (net 2))
+  (segment (start 71.16 74.16) (end 71.1 74.1) (width 0.3) (layer "F.Cu") (net 2))
   (segment (start 119.4 72.4) (end 120.4 72.4) (width 0.3) (layer "F.Cu") (net 2))
   (segment (start 91.05 70.5) (end 92.1 70.5) (width 0.3) (layer "F.Cu") (net 2))
@@
   (via (at 64.8 83.3) (size 0.64) (drill 0.35) (layers "F.Cu" "B.Cu") (net 2))
   (via (at 113.8 118.6) (size 0.64) (drill 0.35) (layers "F.Cu" "B.Cu") (net 2))
+  (via (at 71.1 74.1) (size 0.55) (drill 0.3) (layers "F.Cu" "B.Cu") (net 2))
   (via (at 111.7 78.9) (size 0.64) (drill 0.35) (layers "F.Cu" "B.Cu") (net 2))
   (via (at 96.5 77.2) (size 0.64) (drill 0.35) (layers "F.Cu" "B.Cu") (net 2))
@@
   (via (at 106.4 76.6) (size 0.55) (drill 0.25) (layers "F.Cu" "B.Cu") (net 24))
   (segment (start 106.4 76.6) (end 106.4 70.5) (width 0.15) (layer "B.Cu") (net 24))
-  (segment (start 72.7 72.915) (end 72.725 72.89) (width 0.15) (layer "F.Cu") (net 25))
-  (segment (start 72.725 73.525) (end 72.7 73.5) (width 0.15) (layer "F.Cu") (net 25))
-  (segment (start 75.63 75.43) (end 77.675 75.43) (width 0.15) (layer "F.Cu") (net 25))
   (segment (start 72.59 66.31) (end 72.7 66.2) (width 0.15) (layer "F.Cu") (net 25))
+  (segment (start 72.725 72.89) (end 72.725 71.925) (width 0.15) (layer "F.Cu") (net 25))
+  (segment (start 72.725 71.925) (end 72.7 71.9) (width 0.15) (layer "F.Cu") (net 25))
+  (segment (start 77.675 75.43) (end 75.93 75.43) (width 0.15) (layer "F.Cu") (net 25))
+  (segment (start 75.93 75.43) (end 73.39 72.89) (width 0.15) (layer "F.Cu") (net 25))
   (segment (start 63.95 66.31) (end 72.59 66.31) (width 0.15) (layer "F.Cu") (net 25))
-  (segment (start 72.7 73.5) (end 72.7 72.915) (width 0.15) (layer "F.Cu") (net 25))
-  (segment (start 72.725 74.16) (end 74.36 74.16) (width 0.15) (layer "F.Cu") (net 25))
-  (segment (start 74.36 74.16) (end 75.63 75.43) (width 0.15) (layer "F.Cu") (net 25))
-  (segment (start 72.725 74.16) (end 72.725 73.525) (width 0.15) (layer "F.Cu") (net 25))
+  (segment (start 73.39 72.89) (end 72.725 72.89) (width 0.15) (layer "F.Cu") (net 25))
   (via (at 72.7 66.2) (size 0.55) (drill 0.25) (layers "F.Cu" "B.Cu") (net 25))
-  (via (at 72.7 73.5) (size 0.55) (drill 0.25) (layers "F.Cu" "B.Cu") (net 25))
-  (segment (start 72.7 66.2) (end 72.7 73.5) (width 0.15) (layer "B.Cu") (net 25))
+  (via (at 72.7 71.9) (size 0.55) (drill 0.3) (layers "F.Cu" "B.Cu") (net 25))
+  (segment (start 72.7 71.9) (end 72.7 66.2) (width 0.15) (layer "B.Cu") (net 25))
   (segment (start 75.4 74.1) (end 77.615 74.1) (width 0.15) (layer "F.Cu") (net 26))
   (segment (start 63.95 68.85) (end 75.25 68.85) (width 0.15) (layer "F.Cu") (net 26))
